File: krtkl-breakybreaky-hdmi-expansion.sch (KiCad schematic (older format))
At the start: 39 parts, among them J1 SMH-120-02-T-D, J2 685119134923, J3 solder_jumper, Q1 BSS138AKA, Q2 BSS138AKA, Q3 BSS138AKA, U1 TPD12S016PWR, U2 TPS61232DRCT

Commit message: Finished routing, minor footprint fixes
Parts:
- FB1: footprint antmicro-footprints:0603 -> antmicro-footprints:0603-res
Changed lines of the file:
@@
-	1    0    0    -1
-$EndComp
-$Comp
-L antmicroFerriteBeadsandChips:BLM18PG121SN1D FB1
-U 1 1 5E6A7299
-P 4150 3500
-F 0 "FB1" H 4150 3750 60  0000 C CNN
-F 1 "BLM18PG121SN1D" H 4150 3650 60  0000 C CNN
-F 2 "antmicro-footprints:0603" H 4350 3700 60  0001 L CNN
-F 3 "https://www.murata.com/en-us/products/productdata/8796738650142/ENFA0003.pdf" H 4350 3800 60  0001 L CNN
-F 4 "BLM18PG121SN1D" H 4350 4000 60  0001 L CNN "MPN"
-F 5 "Murata Electronics North America" H 4350 4600 60  0001 L CNN "Manufacturer"
-	1    4150 3500
 	1    0    0    -1
 $EndComp
@@
 	1    0    0    -1
 $EndComp
+$Comp
+L antmicroFerriteBeadsandChips:BLM18PG121SN1D FB1
+U 1 1 5ED64AD2
+P 4150 3500
+F 0 "FB1" H 4150 3787 60  0000 C CNN
+F 1 "BLM18PG121SN1D" H 4150 3681 60  0000 C CNN
+F 2 "antmicro-footprints:0603-res" H 4350 3700 60  0001 L CNN
+F 3 "https://www.murata.com/en-us/products/productdata/8796738650142/ENFA0003.pdf" H 4350 3800 60  0001 L CNN
+F 4 "BLM18PG121SN1D" H 4350 4000 60  0001 L CNN "MPN"
+F 5 "Murata Electronics North America" H 4350 4600 60  0001 L CNN "Manufacturer"
+	1    4150 3500
+	1    0    0    -1
+$EndComp

Commit message: Added logotypes
Parts:
- removed SHIELD (x2): Earth, symbol power:Earth
Connections:
- net labels added: Earth
Other:
- note added: "HPD negation"
- note removed: "TODO: Check orientation and pinout before routing"
- note removed: "TODO: add schematic sections, add logotypes and branding\n"
- moved on the sheet: J2

Commit message: Added testpads, 0R on EDID and board branding to PCB
Parts:
- added R13, R14: R_0R_0402, antmicro-footprints:0402-res, symbol antmicroResistors0402:R_0R_0402
- added TP1, TP2, TP3, TP4, TP5, TP6: TP_SMD1MM, antmicro-footprints:Testpoint_smd_1mm, symbol antmicroTestPoints:TP_SMD1MM
- 3V3, 5V0, LED1, LED2: footprint antmicro-footprints:LED_0603 -> krtkl-breakybreaky-hdmi-expansion-footprints:LED_0603; symbol antmicroLEDIndicationDiscrete:KP-1608CGCK -> krtkl-breakybreaky-hdmi-expansion:KP-1608CGCK
- C1, C2, C3: footprint antmicro-footprints:0402-cap -> krtkl-breakybreaky-hdmi-expansion-footprints:0402-cap; symbol antmicroCapacitors0402:C_100n_0402_6V3 -> krtkl-breakybreaky-hdmi-expansion:C_100n_0402_6V3
- C4: footprint antmicro-footprints:0805-cap -> krtkl-breakybreaky-hdmi-expansion-footprints:0805-cap; symbol antmicroCapacitorsmisc:C_22u_0805 -> krtkl-breakybreaky-hdmi-expansion:C_22u_0805
- C5: footprint antmicro-footprints:0402-cap -> krtkl-breakybreaky-hdmi-expansion-footprints:0402-cap; symbol antmicroCapacitors0402:C_10n_0402 -> krtkl-breakybreaky-hdmi-expansion:C_10n_0402
- C6, C7, C8: footprint antmicro-footprints:0805-cap -> krtkl-breakybreaky-hdmi-expansion-footprints:0805-cap; symbol antmicroCapacitorsmisc:C_22u_0805_10V -> krtkl-breakybreaky-hdmi-expansion:C_22u_0805_10V
- D1: footprint antmicro-footprints:SOD-323F -> krtkl-breakybreaky-hdmi-expansion-footprints:SOD-323F; symbol antmicroDiodesRectifiersSingle:1N4148WS -> krtkl-breakybreaky-hdmi-expansion:1N4148WS
- FB1: footprint antmicro-footprints:0603-res -> krtkl-breakybreaky-hdmi-expansion-footprints:0603-res; symbol antmicroFerriteBeadsandChips:BLM18PG121SN1D -> krtkl-breakybreaky-hdmi-expansion:BLM18PG121SN1D
- J1: footprint antmicro-footprints:SMH-120-02-T-D -> krtkl-breakybreaky-hdmi-expansion-footprints:SMH-120-02-T-D; symbol antmicroRectangularConnectorsHeadersFemalePins:SMH-120-02-T-D -> krtkl-breakybreaky-hdmi-expansion:SMH-120-02-T-D
- J2: footprint antmicro-footprints:HDMI_A_Female_685119134923 -> krtkl-breakybreaky-hdmi-expansion-footprints:HDMI_A_Female_685119134923; symbol antmicroUSBDVIHDMIConnectors:685119134923 -> krtkl-breakybreaky-hdmi-expansion:685119134923
- J3: footprint antmicro-footprints:SolderJumper-0.6x1.4mm -> krtkl-breakybreaky-hdmi-expansion-footprints:SolderJumper-0.6x1.4mm; symbol antmicroShuntsJumpers:solder_jumper -> krtkl-breakybreaky-hdmi-expansion:solder_jumper
- L1: footprint antmicro-footprints:XFL4020-102MEB -> krtkl-breakybreaky-hdmi-expansion-footprints:XFL4020-102MEB; symbol antmicroFixedInductors:XFL4020-102MEB -> krtkl-breakybreaky-hdmi-expansion:XFL4020-102MEB
- N1: footprint antmicro-footprints:oshw-logo -> krtkl-breakybreaky-hdmi-expansion-footprints:oshw-logo; symbol antmicroMechanicalParts:oshw_logo -> krtkl-breakybreaky-hdmi-expansion:oshw_logo
- N2: footprint antmicro-footprints:antmicro-logo_scaled_20mm -> krtkl-breakybreaky-hdmi-expansion-footprints:antmicro-logo_scaled_20mm; symbol antmicroMechanicalParts:antmicro_logo -> krtkl-breakybreaky-hdmi-expansion:antmicro_logo
- Q1, Q2, Q3: footprint antmicro-footprints:SOT-23-3 -> krtkl-breakybreaky-hdmi-expansion-footprints:SOT-23-3; symbol antmicroTransistorsFETsMOSFETsSingle:BSS138AKA -> krtkl-breakybreaky-hdmi-expansion:BSS138AKA
- R1, R2, R4: footprint antmicro-footprints:0402-res -> krtkl-breakybreaky-hdmi-expansion-footprints:0402-res; symbol antmicroResistors0402:R_10k_0402 -> krtkl-breakybreaky-hdmi-expansion:R_10k_0402
- R10: footprint antmicro-footprints:0402-res -> krtkl-breakybreaky-hdmi-expansion-footprints:0402-res; symbol antmicroResistors0402:R_402k_0402 -> krtkl-breakybreaky-hdmi-expansion:R_402k_0402
- R11: footprint antmicro-footprints:0402-res -> krtkl-breakybreaky-hdmi-expansion-footprints:0402-res; symbol antmicroResistors0402:R_100k_0402 -> krtkl-breakybreaky-hdmi-expansion:R_100k_0402
- R12: footprint antmicro-footprints:0603-res -> krtkl-breakybreaky-hdmi-expansion-footprints:0603-res; symbol antmicroResistors0603:R_0R_0603 -> krtkl-breakybreaky-hdmi-expansion:R_0R_0603
- R3: footprint antmicro-footprints:0402-res -> krtkl-breakybreaky-hdmi-expansion-footprints:0402-res; symbol antmicroResistors0402:R_0R_0402 -> krtkl-breakybreaky-hdmi-expansion:R_0R_0402
- R5: footprint antmicro-footprints:0402-res -> krtkl-breakybreaky-hdmi-expansion-footprints:0402-res; symbol antmicroResistors0402:R_470R_0402 -> krtkl-breakybreaky-hdmi-expansion:R_470R_0402
- R6, R7, R8: footprint antmicro-footprints:0402-res -> krtkl-breakybreaky-hdmi-expansion-footprints:0402-res; symbol antmicroResistors0402:R_330R_0402 -> krtkl-breakybreaky-hdmi-expansion:R_330R_0402
- R9: footprint antmicro-footprints:0603-res -> krtkl-breakybreaky-hdmi-expansion-footprints:0603-res; symbol antmicroResistors0603:R_1M_0603 -> krtkl-breakybreaky-hdmi-expansion:R_1M_0603
- U1: footprint antmicro-footprints:TPD12S016PWR -> krtkl-breakybreaky-hdmi-expansion-footprints:TPD12S016PWR; symbol antmicroInterfaceControllers:TPD12S016PWR -> krtkl-breakybreaky-hdmi-expansion:TPD12S016PWR
- U2: footprint antmicro-footprints:VSON-10-1EP_3x3mm -> krtkl-breakybreaky-hdmi-expansion-footprints:VSON-10-1EP_3x3mm; symbol antmicroDCDCConverters:TPS61232DRCT -> krtkl-breakybreaky-hdmi-expansion:TPS61232DRCT
Connections:
- wire segments 190 -> 192
Other:
- note added: "T20"
- note added: "U20"
- note added: "V20"
- note added: "W20"

Commit message: Updated documentation, added README and LICENSE
Parts:
- R13, R14: footprint antmicro-footprints:0402-res -> krtkl-breakybreaky-hdmi-expansion-footprints:0402-res; symbol antmicroResistors0402:R_0R_0402 -> krtkl-breakybreaky-hdmi-expansion:R_0R_0402
- TP1, TP2, TP3, TP4, TP5, TP6: footprint antmicro-footprints:Testpoint_smd_1mm -> krtkl-breakybreaky-hdmi-expansion-footprints:Testpoint_smd_1mm; symbol antmicroTestPoints:TP_SMD1MM -> krtkl-breakybreaky-hdmi-expansion:TP_SMD1MM
Changed lines of the file:
@@
 HDMI_SCL_3V3
 $Comp
-L antmicroTestPoints:TP_SMD1MM TP5
+L krtkl-breakybreaky-hdmi-expansion:TP_SMD1MM TP5
 U 1 1 5E685C64
 P 12200 7300
 F 0 "TP5" V 12150 7300 50  0000 R CNN
 F 1 "TP_SMD1MM" H 12200 7200 50  0001 C CNN
-F 2 "antmicro-footprints:Testpoint_smd_1mm" H 12400 7500 60  0001 L CNN
+F 2 "krtkl-breakybreaky-hdmi-expansion-footprints:Testpoint_smd_1mm" H 12400 7500 60  0001 L CNN
 F 3 "" H 12400 7600 60  0001 L CNN
 	1    12200 7300
@@
 $EndComp
 $Comp
-L antmicroTestPoints:TP_SMD1MM TP6
+L krtkl-breakybreaky-hdmi-expansion:TP_SMD1MM TP6
 U 1 1 5E68AC0C
 P 12200 7400
 F 0 "TP6" V 12250 7400 50  0000 R CNN
 F 1 "TP_SMD1MM" H 12200 7300 50  0001 C CNN
-F 2 "antmicro-footprints:Testpoint_smd_1mm" H 12400 7600 60  0001 L CNN
+F 2 "krtkl-breakybreaky-hdmi-expansion-footprints:Testpoint_smd_1mm" H 12400 7600 60  0001 L CNN
 F 3 "" H 12400 7700 60  0001 L CNN
 	1    12200 7400
@@
 $EndComp
 $Comp
-L antmicroResistors0402:R_0R_0402 R14
+L krtkl-breakybreaky-hdmi-expansion:R_0R_0402 R14
 U 1 1 5E6C715E
 P 13500 7300
 F 0 "R14" H 13350 7350 60  0000 C CNN
 F 1 "R_0R_0402" H 13500 7150 60  0001 C CNN
-F 2 "antmicro-footprints:0402-res" H 13700 7500 60  0001 L CNN
+F 2 "krtkl-breakybreaky-hdmi-expansion-footprints:0402-res" H 13700 7500 60  0001 L CNN
 F 3 "" H 13500 7300 50  0001 C CNN
 F 4 "PANASONIC" H 13700 7700 60  0001 L CNN "Manufacturer"
@@
 	13350 7300 12300 7300
 $Comp
-L antmicroResistors0402:R_0R_0402 R13
+L krtkl-breakybreaky-hdmi-expansion:R_0R_0402 R13
 U 1 1 5E6C7819
 P 13150 7400
 F 0 "R13" H 13000 7450 60  0000 C CNN
 F 1 "R_0R_0402" H 13150 7250 60  0001 C CNN
-F 2 "antmicro-footprints:0402-res" H 13350 7600 60  0001 L CNN
+F 2 "krtkl-breakybreaky-hdmi-expansion-footprints:0402-res" H 13350 7600 60  0001 L CNN
 F 3 "" H 13150 7400 50  0001 C CNN
 F 4 "PANASONIC" H 13350 7800 60  0001 L CNN "Manufacturer"
@@
 	12300 7400 13000 7400
 $Comp
-L antmicroTestPoints:TP_SMD1MM TP1
+L krtkl-breakybreaky-hdmi-expansion:TP_SMD1MM TP1
 U 1 1 5E74470E
 P 2650 7250
 F 0 "TP1" V 2600 7250 50  0000 R CNN
 F 1 "TP_SMD1MM" H 2650 7150 50  0001 C CNN
-F 2 "antmicro-footprints:Testpoint_smd_1mm" H 2850 7450 60  0001 L CNN
+F 2 "krtkl-breakybreaky-hdmi-expansion-footprints:Testpoint_smd_1mm" H 2850 7450 60  0001 L CNN
 F 3 "" H 2850 7550 60  0001 L CNN
 	1    2650 7250
@@
 $EndComp
 $Comp
-L antmicroTestPoints:TP_SMD1MM TP2
+L krtkl-breakybreaky-hdmi-expansion:TP_SMD1MM TP2
 U 1 1 5E7450D0
 P 2650 7350
 F 0 "TP2" V 2600 7350 50  0000 R CNN
 F 1 "TP_SMD1MM" H 2650 7250 50  0001 C CNN
-F 2 "antmicro-footprints:Testpoint_smd_1mm" H 2850 7550 60  0001 L CNN
+F 2 "krtkl-breakybreaky-hdmi-expansion-footprints:Testpoint_smd_1mm" H 2850 7550 60  0001 L CNN
 F 3 "" H 2850 7650 60  0001 L CNN
 	1    2650 7350
@@
 $EndComp
 $Comp
-L antmicroTestPoints:TP_SMD1MM TP3
+L krtkl-breakybreaky-hdmi-expansion:TP_SMD1MM TP3
 U 1 1 5E745357
 P 2650 7550
 F 0 "TP3" V 2600 7550 50  0000 R CNN
 F 1 "TP_SMD1MM" H 2650 7450 50  0001 C CNN
-F 2 "antmicro-footprints:Testpoint_smd_1mm" H 2850 7750 60  0001 L CNN
+F 2 "krtkl-breakybreaky-hdmi-expansion-footprints:Testpoint_smd_1mm" H 2850 7750 60  0001 L CNN
 F 3 "" H 2850 7850 60  0001 L CNN
 	1    2650 7550
@@
 $EndComp
 $Comp
-L antmicroTestPoints:TP_SMD1MM TP4
+L krtkl-breakybreaky-hdmi-expansion:TP_SMD1MM TP4
 U 1 1 5E7456DD
 P 2650 7650
 F 0 "TP4" V 2600 7650 50  0000 R CNN
 F 1 "TP_SMD1MM" H 2650 7550 50  0001 C CNN
-F 2 "antmicro-footprints:Testpoint_smd_1mm" H 2850 7850 60  0001 L CNN
+F 2 "krtkl-breakybreaky-hdmi-expansion-footprints:Testpoint_smd_1mm" H 2850 7850 60  0001 L CNN
 F 3 "" H 2850 7950 60  0001 L CNN
 	1    2650 7650
