File: snickerdoodle-hdmi-breakout.sch (KiCad schematic (older format))
At the start: 45 parts, among them J1 SMH-120-02-T-D, J2 685119134923, J3 solder_jumper, Q1 BSS138AKA, Q2 BSS138AKA, Q3 BSS138AKA, U1 TPD12S016PWR, U2 TPS61232DRCT

Commit message: Updated component library
Parts:
- 3V3, 5V0, LED1, LED2: footprint krtkl-breakybreaky-hdmi-expansion-footprints:LED_0603 -> snickerdoodle-hdmi-breakout-footprints:LED_0603; symbol krtkl-breakybreaky-hdmi-expansion:KP-1608CGCK -> snickerdoodle-hdmi-breakout:KP-1608CGCK
- C1, C2, C3: footprint krtkl-breakybreaky-hdmi-expansion-footprints:0402-cap -> snickerdoodle-hdmi-breakout-footprints:0402-cap; symbol krtkl-breakybreaky-hdmi-expansion:C_100n_0402_6V3 -> snickerdoodle-hdmi-breakout:C_100n_0402_6V3
- C4: footprint krtkl-breakybreaky-hdmi-expansion-footprints:0805-cap -> snickerdoodle-hdmi-breakout-footprints:0805-cap; symbol krtkl-breakybreaky-hdmi-expansion:C_22u_0805 -> snickerdoodle-hdmi-breakout:C_22u_0805
- C5: footprint krtkl-breakybreaky-hdmi-expansion-footprints:0402-cap -> snickerdoodle-hdmi-breakout-footprints:0402-cap; symbol krtkl-breakybreaky-hdmi-expansion:C_10n_0402 -> snickerdoodle-hdmi-breakout:C_10n_0402
- C6, C7, C8: footprint krtkl-breakybreaky-hdmi-expansion-footprints:0805-cap -> snickerdoodle-hdmi-breakout-footprints:0805-cap; symbol krtkl-breakybreaky-hdmi-expansion:C_22u_0805_10V -> snickerdoodle-hdmi-breakout:C_22u_0805_10V
- D1: footprint krtkl-breakybreaky-hdmi-expansion-footprints:SOD-323F -> snickerdoodle-hdmi-breakout-footprints:SOD-323F; symbol krtkl-breakybreaky-hdmi-expansion:1N4148WS -> snickerdoodle-hdmi-breakout:1N4148WS
- FB1: footprint krtkl-breakybreaky-hdmi-expansion-footprints:0603-res -> snickerdoodle-hdmi-breakout-footprints:0603-res; symbol krtkl-breakybreaky-hdmi-expansion:BLM18PG121SN1D -> snickerdoodle-hdmi-breakout:BLM18PG121SN1D; Manufacturer Murata Electronics North America -> Murata Electronics North America
- J1: footprint krtkl-breakybreaky-hdmi-expansion-footprints:SMH-120-02-T-D -> snickerdoodle-hdmi-breakout-footprints:SMH-120-02-T-D; symbol krtkl-breakybreaky-hdmi-expansion:SMH-120-02-T-D -> snickerdoodle-hdmi-breakout:SMH-120-02-T-D
- J2: footprint krtkl-breakybreaky-hdmi-expansion-footprints:HDMI_A_Female_685119134923 -> snickerdoodle-hdmi-breakout-footprints:HDMI_A_Female_685119134923; symbol krtkl-breakybreaky-hdmi-expansion:685119134923 -> snickerdoodle-hdmi-breakout:685119134923
- J3: footprint krtkl-breakybreaky-hdmi-expansion-footprints:SolderJumper-0.6x1.4mm -> snickerdoodle-hdmi-breakout-footprints:SolderJumper-0.6x1.4mm; symbol krtkl-breakybreaky-hdmi-expansion:solder_jumper -> snickerdoodle-hdmi-breakout:solder_jumper
- L1: footprint krtkl-breakybreaky-hdmi-expansion-footprints:XFL4020-102MEB -> snickerdoodle-hdmi-breakout-footprints:XFL4020-102MEB; symbol krtkl-breakybreaky-hdmi-expansion:XFL4020-102MEB -> snickerdoodle-hdmi-breakout:XFL4020-102MEB
- N1: footprint krtkl-breakybreaky-hdmi-expansion-footprints:oshw-logo -> snickerdoodle-hdmi-breakout-footprints:oshw-logo; symbol krtkl-breakybreaky-hdmi-expansion:oshw_logo -> snickerdoodle-hdmi-breakout:oshw_logo
- N2: footprint krtkl-breakybreaky-hdmi-expansion-footprints:antmicro-logo_scaled_20mm -> snickerdoodle-hdmi-breakout-footprints:antmicro-logo_scaled_20mm; symbol krtkl-breakybreaky-hdmi-expansion:antmicro_logo -> snickerdoodle-hdmi-breakout:antmicro_logo
- Q1, Q2, Q3: footprint krtkl-breakybreaky-hdmi-expansion-footprints:SOT-23-3 -> snickerdoodle-hdmi-breakout-footprints:SOT-23-3; symbol krtkl-breakybreaky-hdmi-expansion:BSS138AKA -> snickerdoodle-hdmi-breakout:BSS138AKA
- R1, R2, R4: footprint krtkl-breakybreaky-hdmi-expansion-footprints:0402-res -> snickerdoodle-hdmi-breakout-footprints:0402-res; symbol krtkl-breakybreaky-hdmi-expansion:R_10k_0402 -> snickerdoodle-hdmi-breakout:R_10k_0402
- R10: footprint krtkl-breakybreaky-hdmi-expansion-footprints:0402-res -> snickerdoodle-hdmi-breakout-footprints:0402-res; symbol krtkl-breakybreaky-hdmi-expansion:R_402k_0402 -> snickerdoodle-hdmi-breakout:R_402k_0402
- R11: footprint krtkl-breakybreaky-hdmi-expansion-footprints:0402-res -> snickerdoodle-hdmi-breakout-footprints:0402-res; symbol krtkl-breakybreaky-hdmi-expansion:R_100k_0402 -> snickerdoodle-hdmi-breakout:R_100k_0402
- R12: footprint krtkl-breakybreaky-hdmi-expansion-footprints:0603-res -> snickerdoodle-hdmi-breakout-footprints:0603-res; symbol krtkl-breakybreaky-hdmi-expansion:R_0R_0603 -> snickerdoodle-hdmi-breakout:R_0R_0603
- R13, R14, R3: footprint krtkl-breakybreaky-hdmi-expansion-footprints:0402-res -> snickerdoodle-hdmi-breakout-footprints:0402-res; symbol krtkl-breakybreaky-hdmi-expansion:R_0R_0402 -> snickerdoodle-hdmi-breakout:R_0R_0402
- R5: footprint krtkl-breakybreaky-hdmi-expansion-footprints:0402-res -> snickerdoodle-hdmi-breakout-footprints:0402-res; symbol krtkl-breakybreaky-hdmi-expansion:R_470R_0402 -> snickerdoodle-hdmi-breakout:R_470R_0402
- R6, R7, R8: footprint krtkl-breakybreaky-hdmi-expansion-footprints:0402-res -> snickerdoodle-hdmi-breakout-footprints:0402-res; symbol krtkl-breakybreaky-hdmi-expansion:R_330R_0402 -> snickerdoodle-hdmi-breakout:R_330R_0402
- R9: footprint krtkl-breakybreaky-hdmi-expansion-footprints:0603-res -> snickerdoodle-hdmi-breakout-footprints:0603-res; symbol krtkl-breakybreaky-hdmi-expansion:R_1M_0603 -> snickerdoodle-hdmi-breakout:R_1M_0603
- TP1, TP2, TP3, TP4, TP5, TP6: footprint krtkl-breakybreaky-hdmi-expansion-footprints:Testpoint_smd_1mm -> snickerdoodle-hdmi-breakout-footprints:Testpoint_smd_1mm; symbol krtkl-breakybreaky-hdmi-expansion:TP_SMD1MM -> snickerdoodle-hdmi-breakout:TP_SMD1MM
- U1: footprint krtkl-breakybreaky-hdmi-expansion-footprints:TPD12S016PWR -> snickerdoodle-hdmi-breakout-footprints:TPD12S016PWR; symbol krtkl-breakybreaky-hdmi-expansion:TPD12S016PWR -> snickerdoodle-hdmi-breakout:TPD12S016PWR
- U2: footprint krtkl-breakybreaky-hdmi-expansion-footprints:VSON-10-1EP_3x3mm -> snickerdoodle-hdmi-breakout-footprints:VSON-10-1EP_3x3mm; symbol krtkl-breakybreaky-hdmi-expansion:TPS61232DRCT -> snickerdoodle-hdmi-breakout:TPS61232DRCT

Commit message: Release 1.0.1
Parts:
- Q1, R1, R2: DNP (none) -> 1
- U1: footprint snickerdoodle-hdmi-breakout-footprints:TPD12S016PWR -> snickerdoodle-hdmi-expansion-footprints:TPD12S016PWR; MPN (none) -> TPD12S016PWR; Manufacturer (none) -> Texas Instruments
- U2: footprint snickerdoodle-hdmi-breakout-footprints:VSON-10-1EP_3x3mm -> snickerdoodle-hdmi-expansion-footprints:VSON-10-1EP_3x3mm; MPN (none) -> TPS61232DRCT; Manufacturer (none) -> Texas Instruments
Other:
- note added: "DNP"
Changed lines of the file:
@@
 Title "Snickerdoodle HDMI breakout"
 Date "03/2020"
-Rev "1.0"
+Rev "1.0.1"
 Comp ""
 Comment1 "www.antmicro.com"
@@
 F 5 "CRCW040210K0FKEDHP" H 9550 7600 60  0001 L CNN "MPN"
 F 6 "10k" V 9297 7230 50  0000 R CNN "Val"
+F 7 "1" V 9350 7300 50  0001 C CNN "DNP"
 	1    9350 7300
 	0    -1   -1   0
@@
 F 4 "BSS138AKA" H 9950 7500 60  0001 L CNN "MPN"
 F 5 "ON Semiconductor" H 9950 8100 60  0001 L CNN "Manufacturer"
+F 6 "1" H 9750 7000 50  0001 C CNN "DNP"
 	1    9750 7000
 	1    0    0    -1
@@
 F 5 "SAMTEC" H 3550 4100 60  0001 L CNN "Manufacturer"
 	1    3700 6100
-	1    0    0    -1  krtkl-breakybreaky-hdmi-expansi
+	1    0    0    -1
 $EndComp
 $Comp
@@
 F 0 "U1" H 14450 6215 60  0000 C CNN
 F 1 "TPD12S016PWR" H 14450 6124 60  0000 C CNN
-F 2 "snickerdoodle-hdmi-breakout-footprints:TPD12S016PWR" H 14050 6050 50  0001 C CNN
+F 2 "snickerdoodle-hdmi-expansion-footprints:TPD12S016PWR" H 14050 6050 50  0001 C CNN
 F 3 "http://www.ti.com/lit/ds/symlink/tpd12s016.pdf" H 14050 6050 50  0001 C CNN
+F 4 "TPD12S016PWR" H 14050 6050 50  0001 C CNN "MPN"
+F 5 "Texas Instruments" H 14050 6050 50  0001 C CNN "Manufacturer"
 	1    14050 6050
 	1    0    0    -1
@@
 F 0 "U2" H 13650 3465 60  0000 C CNN
 F 1 "TPS61232DRCT" H 13650 3374 60  0000 C CNN
-F 2 "snickerdoodle-hdmi-breakout-footprints:VSON-10-1EP_3x3mm" H 13550 2500 50  0001 C CNN
+F 2 "snickerdoodle-hdmi-expansion-footprints:VSON-10-1EP_3x3mm" H 13550 2500 50  0001 C CNN
 F 3 "http://www.ti.com/lit/ds/symlink/tps61232.pdf" H 13650 2600 50  0001 C CNN
+F 4 "TPS61232DRCT" H 13650 2700 50  0001 C CNN "MPN"
+F 5 "Texas Instruments" H 13650 2700 50  0001 C CNN "Manufacturer"
 	1    13650 2700
 	1    0    0    -1
@@
 F 5 "CRCW040210K0FKEDHP" H 9950 6800 60  0001 L CNN "MPN"
 F 6 "10k" V 9697 6430 50  0000 R CNN "Val"
+F 7 "1" V 9750 6500 50  0001 C CNN "DNP"
 	1    9750 6500
 	0    -1   -1   0
@@
 Text Notes 1500 7650 0    50   ~ 0
 W20
+Text Notes 9850 7200 0    50   ~ 0
+DNP
+Text Notes 9700 6550 1    50   ~ 0
+DNP
+Text Notes 9300 7400 1    50   ~ 0
+DNP
 $EndSCHEMATC

Commit message: Updated Manufacturer for HDMI connector
Parts:
- J2: footprint snickerdoodle-hdmi-breakout-footprints:HDMI_A_Female_685119134923 -> snickerdoodle-hdmi-expansion-footprints:HDMI_A_Female_685119134923; Manufacturer Amphenol -> Wurth Elektronik
Changed lines of the file:
@@
 F 0 "J2" H 2750 3287 60  0000 C CNN
 F 1 "685119134923" H 2750 3181 60  0000 C CNN
-F 2 "snickerdoodle-hdmi-breakout-footprints:HDMI_A_Female_685119134923" H 2950 2550 60  0001 L CNN
-F 3 "https://en.wikipedia.org/wiki/HDMI" H 2950 2650 60  0001 L CNN
+F 2 "snickerdoodle-hdmi-expansion-footprints:HDMI_A_Female_685119134923" H 2950 2550 60  0001 L CNN
+F 3 "https://www.farnell.com/cad/1641702.pdf?_ga=2.75511573.1630328358.1571653391-156563690.1566371002&_gac=1.138144260.1570692453.EAIaIQobChMIsbyuq5WR5QIVhKiaCh1YMAxzEAYYBiABEgKWa_D_BwE" H 2950 2650 60  0001 L CNN
 F 4 "685119134923" H 2950 2850 60  0001 L CNN "MPN"
-F 5 "Amphenol" H 2950 3450 60  0001 L CNN "Manufacturer"
+F 5 "Wurth Elektronik" H 2950 3450 60  0001 L CNN "Manufacturer"
 	1    2750 2350
 	1    0    0    -1

Commit message: Prepared files for revision 1.1.0 - rotated HDMI connector, changed PCB size
Parts:
- removed J2: 685119134923, snickerdoodle-hdmi-expansion-footprints:HDMI_A_Female_685119134923, symbol snickerdoodle-hdmi-breakout:685119134923
- added J2: 685119134923, antmicro-footprints:HDMI_A_Female_685119134923, symbol antmicroUSBDVIHDMIConnectors:685119134923
Changed lines of the file:
@@
 EESchema Schematic File Version 4
-EELAYER 30 0
+LIBS:snickerdoodle-hdmi-breakout-cache
+EELAYER 26 0
 EELAYER END
 $Descr A3 16535 11693
@@
 V18
 $Comp
-L snickerdoodle-hdmi-breakout:685119134923 J2
-U 1 1 5E64A095
-P 2750 2350
-F 0 "J2" H 2750 3287 60  0000 C CNN
-F 1 "685119134923" H 2750 3181 60  0000 C CNN
-F 2 "snickerdoodle-hdmi-expansion-footprints:HDMI_A_Female_685119134923" H 2950 2550 60  0001 L CNN
-F 3 "https://www.farnell.com/cad/1641702.pdf?_ga=2.75511573.1630328358.1571653391-156563690.1566371002&_gac=1.138144260.1570692453.EAIaIQobChMIsbyuq5WR5QIVhKiaCh1YMAxzEAYYBiABEgKWa_D_BwE" H 2950 2650 60  0001 L CNN
-F 4 "685119134923" H 2950 2850 60  0001 L CNN "MPN"
-F 5 "Wurth Elektronik" H 2950 3450 60  0001 L CNN "Manufacturer"
-	1    2750 2350
-	1    0    0    -1
-$EndComp
-$Comp
 L snickerdoodle-hdmi-breakout:BLM18PG121SN1D FB1
 U 1 1 5ED64AD2
@@
 Text Notes 9300 7400 1    50   ~ 0
 DNP
+$Comp
+L antmicroUSBDVIHDMIConnectors:685119134923 J2
+U 1 1 5E7AA1A0
+P 2750 2350
+F 0 "J2" H 2750 3287 60  0000 C CNN
+F 1 "685119134923" H 2750 3181 60  0000 C CNN
+F 2 "antmicro-footprints:HDMI_A_Female_685119134923" H 2950 2550 60  0001 L CNN
+F 3 "https://www.farnell.com/cad/1641702.pdf?_ga=2.75511573.1630328358.1571653391-156563690.1566371002&_gac=1.138144260.1570692453.EAIaIQobChMIsbyuq5WR5QIVhKiaCh1YMAxzEAYYBiABEgKWa_D_BwE" H 2950 2650 60  0001 L CNN
+F 4 "685119134923" H 2950 2850 60  0001 L CNN "MPN"
+F 5 "Amphenol" H 2950 3450 60  0001 L CNN "Manufacturer"
+	1    2750 2350
+	1    0    0    -1
+$EndComp
 $EndSCHEMATC
