File: snickerdoodle-hdmi-breakout.sch (KiCad schematic (older format))
At the start: 45 parts, among them J1 SMH-120-02-T-D, J2 685119134923, J3 solder_jumper, Q1 BSS138AKA, Q2 BSS138AKA, Q3 BSS138AKA, U1 TPD12S016PWR, U2 TPS61232DRCT

Commit message: Changed R10, re-generated documentation
Parts:
- removed R10: R_402k_0402, snickerdoodle-hdmi-breakout-footprints:0402-res, symbol snickerdoodle-hdmi-breakout:R_402k_0402
- added R10: R_0R_0402, snickerdoodle-hdmi-breakout-footprints:0402-res, symbol snickerdoodle-hdmi-breakout:R_0R_0402
- J2: footprint antmicro-footprints:HDMI_A_Female_685119134923 -> snickerdoodle-hdmi-breakout-footprints:HDMI_A_Female_685119134923; symbol antmicroUSBDVIHDMIConnectors:685119134923 -> snickerdoodle-hdmi-breakout:685119134923
Changed lines of the file:
@@
-	0    1    1    0
-$EndComp
-$Comp
-L snickerdoodle-hdmi-breakout:R_402k_0402 R10
-U 1 1 5E8DBEE3
-P 14400 2650
-F 0 "R10" V 14355 2720 60  0000 L CNN
-F 1 "R_402k_0402" H 14400 2500 60  0001 C CNN
-F 2 "snickerdoodle-hdmi-breakout-footprints:0402-res" H 14600 2850 60  0001 L CNN
-F 3 "" H 14400 2650 50  0001 C CNN
-F 4 "VISHAY" H 14600 3050 60  0001 L CNN "Manufacturer"
-F 5 "CRCW0402402KFKED" H 14600 2950 60  0001 L CNN "MPN"
-F 6 "402k" V 14453 2720 50  0000 L CNN "Val"
-	1    14400 2650
 	0    1    1    0
 $EndComp
@@
 DNP
 $Comp
-L antmicroUSBDVIHDMIConnectors:685119134923 J2
+L snickerdoodle-hdmi-breakout:685119134923 J2
 U 1 1 5E7AA1A0
 P 2750 2350
 F 0 "J2" H 2750 3287 60  0000 C CNN
 F 1 "685119134923" H 2750 3181 60  0000 C CNN
-F 2 "antmicro-footprints:HDMI_A_Female_685119134923" H 2950 2550 60  0001 L CNN
+F 2 "snickerdoodle-hdmi-breakout-footprints:HDMI_A_Female_685119134923" H 2950 2550 60  0001 L CNN
 F 3 "https://www.farnell.com/cad/1641702.pdf?_ga=2.75511573.1630328358.1571653391-156563690.1566371002&_gac=1.138144260.1570692453.EAIaIQobChMIsbyuq5WR5QIVhKiaCh1YMAxzEAYYBiABEgKWa_D_BwE" H 2950 2650 60  0001 L CNN
 F 4 "685119134923" H 2950 2850 60  0001 L CNN "MPN"
@@
 	1    0    0    -1
 $EndComp
+$Comp
+L snickerdoodle-hdmi-breakout:R_0R_0402 R10
+U 1 1 5E7DBB4E
+P 14400 2650
+F 0 "R10" H 14400 2863 60  0000 C CNN
+F 1 "R_0R_0402" H 14400 2500 60  0001 C CNN
+F 2 "snickerdoodle-hdmi-breakout-footprints:0402-res" H 14600 2850 60  0001 L CNN
+F 3 "" H 14400 2650 50  0001 C CNN
+F 4 "PANASONIC" H 14600 3050 60  0001 L CNN "Manufacturer"
+F 5 "ERJ2GE0R00X" H 14600 2950 60  0001 L CNN "MPN"
+F 6 "0R" H 14400 2765 50  0000 C CNN "Val"
+	1    14400 2650
+	0    1    1    0
+$EndComp
 $EndSCHEMATC
